File: can_middle/can_middle.kicad_pcb (KiCad board)
At the start: 2 copper layers, 7 parts, among them J1 Conn_CAN_IN, J2 Conn_CAN_TAP, J3 Conn_CAN_BRIDGE, U1 CAN_Transceiver, U2 CAN_Transceiver

Commit message: layed out
Parts:
- removed ESP-MASTER1, ESP-SLAVE1: DOIT-ESP32-DEVKIT-V1, doit-esp32-devkit-kicad-master:ESP32-DOIT-DEVKIT
- added J4: Conn_01x02, Connector_JST:JST_EH_B2B-EH-A_1x02_P2.50mm_Vertical, F.Cu at (185.4, 81.3)
- added U3: ESP32_master, footprints:esp32_devkit_v1_doit, F.Cu at (182.9, 127.6)
- added U4: ESP32_slave, footprints:esp32_devkit_v1_doit, F.Cu at (149.9, 127.6)
- added U5: dcBuck, footprints:dcbuck, F.Cu at (170.2, 83.8)
- J1, J2, J3: footprint Connector_IDC:IDC-Header_2x10_P2.54mm_Vertical -> Connector_PinHeader_2.54mm:PinHeader_2x10_P2.54mm_Vertical
- moved J3 62.8 mm to (139.7, 91.4), turned to 180 degrees
- moved J1 45.8 mm to (195.6, 91.4), turned to 180 degrees
- moved U1 35.9 mm to (170.2, 108.0)
- moved U2 30.4 mm to (137.2, 108.0)
- moved J2 26.4 mm to (156.2, 91.4), turned to 180 degrees
Routing:
- net /a11_EXT_CANH: track 0.00 -> 83.7 mm
- net /a12_EXT_CANL: track 0.00 -> 78.3 mm
- net /a17: track 0.00 -> 57.9 mm, vias 0 -> 1
- net /a7: track 0.00 -> 57.9 mm
- net /a1: track 0.00 -> 57.8 mm
- net /a4: track 0.00 -> 57.8 mm
- net /a3: track 0.00 -> 57.8 mm
- net /a2: track 0.00 -> 57.8 mm
- net /b11_EXT_CANH: track 0.00 -> 46.9 mm
- net /b12_EXT_CANL: track 0.00 -> 45.4 mm
- net /MASTER_CAN_TX: track 0.00 -> 43.4 mm
- net /SLAVE_CAN_TX: track 0.00 -> 43.4 mm
- net /SLAVE_CAN_RX: track 0.00 -> 38.3 mm
- net /MASTER_CAN_RX: track 0.00 -> 38.3 mm
- net /MASTER-TX: track 0.00 -> 34.1 mm
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- added copper zone on B.Cu, net +3.3V
- added copper zone on F.Cu, net GND
Other:
- board outline added: 73.7 x 116.8 mm

Commit message: cleanups before printing
Parts:
- J2, J3: footprint Connector_PinHeader_2.54mm:PinHeader_2x10_P2.54mm_Vertical -> footprints:VW T20d connector
- U1: value CAN_Transceiver -> CAN_Transceiver tap
- U2: value CAN_Transceiver -> CAN_Transceiver br
Other:
- board text added: "+12V"
- board text added: "GND"
